Commit message: add keyboard commands

File: src/gazebo_sim/racecar_description/urdf/racecar.xacro (robot description, xacro)
@@ -82,5 +82,5 @@
     <child link="left_steering_hinge" />
     <axis xyz="-1 0 0" />
-    <limit lower="-1.0" upper="1.0" effort="10" velocity="100" />
+    <limit lower="-0.5" upper="0.5" effort="10" velocity="100" />
   </joint>
   <xacro:steering_hinge_transmission name="left_steering_hinge" />
@@ -100,5 +100,5 @@
     <child link="right_steering_hinge" />
     <axis xyz="-1 0 0" />
-    <limit lower="-1.0" upper="1.0" effort="10" velocity="100" />
+    <limit lower="-0.5" upper="0.5" effort="10" velocity="100" />
   </joint>
   <xacro:steering_hinge_transmission name="right_steering_hinge" />
