Commit message: Added AWS track and scaled racecar

File: src/simulator/racecar_description/urdf/macros.xacro (robot description, xacro)
@@ -4,22 +4,22 @@
 <xacro:macro name="chassis_inertial_params">
   <origin xyz="0.1477 0 0" rpy="0 0 0" />
-  <mass value="4.0" />
-  <inertia ixx="0.010609" ixy="0"          ixz="0"
-                          iyy="0.050409"   iyz="0"
-                                           izz="0.05865" />
+  <mass value="20.0" />
+  <inertia ixx="0.150609" ixy="0"          ixz="0"
+                          iyy="0.750409"   iyz="0"
+                                           izz="0.75865" />
 </xacro:macro>
 <xacro:macro name="left_wheels_inertial_params">
   <origin xyz="0 0 -0.0225" rpy="0 0 0" />
   <mass value="0.34055" />
-  <inertia ixx="0.00026046" ixy="0"          ixz="0"
-                            iyy="0.00026046" iyz="0"
-                                             izz="0.00041226" />
+  <inertia ixx="0.00066046" ixy="0"          ixz="0"
+                            iyy="0.00066046" iyz="0"
+                                             izz="0.00121226" />
 </xacro:macro>
 <xacro:macro name="right_wheels_inertial_params">
   <origin xyz="0 0 0.0225" rpy="0 0 0" />
   <mass value="0.34055" />
-  <inertia ixx="0.00026046" ixy="0"          ixz="0"
-                            iyy="0.00026046" iyz="0"
-                                             izz="0.00041226" />
+  <inertia ixx="0.00066046" ixy="0"          ixz="0"
+                            iyy="0.00066046" iyz="0"
+                                             izz="0.00121226" />
 </xacro:macro>
 <xacro:macro name="steering_hinge_inertial_params">
@@ -41,5 +41,5 @@
   <origin xyz="0 0 0" rpy="0 0 0" />
   <geometry>
-    <mesh filename="package://racecar_description/meshes/chassis.STL" />
+    <mesh filename="package://racecar_description/meshes/chassis.STL" scale="3 3 3" />
   </geometry>
 </xacro:macro>
@@ -47,5 +47,5 @@
   <origin xyz="0 0 0" rpy="0 0 0" />
   <geometry>
-    <mesh filename="package://racecar_description/meshes/left_rear_wheel.STL" />
+    <mesh filename="package://racecar_description/meshes/left_rear_wheel.STL" scale="3 3 3" />
   </geometry>
 </xacro:macro>
@@ -53,5 +53,5 @@
   <origin xyz="0 0 0" rpy="0 0 0" />
   <geometry>
-    <mesh filename="package://racecar_description/meshes/right_rear_wheel.STL" />
+    <mesh filename="package://racecar_description/meshes/right_rear_wheel.STL" scale="3 3 3"/>
   </geometry>
 </xacro:macro>
@@ -59,5 +59,5 @@
   <origin xyz="0 0 0" rpy="0 0 0" />
   <geometry>
-    <mesh filename="package://racecar_description/meshes/left_front_wheel.STL" />
+    <mesh filename="package://racecar_description/meshes/left_front_wheel.STL" scale="3 3 3"/>
   </geometry>
 </xacro:macro>
@@ -65,5 +65,5 @@
   <origin xyz="0 0 0" rpy="0 0 0" />
   <geometry>
-    <mesh filename="package://racecar_description/meshes/right_front_wheel.STL" />
+    <mesh filename="package://racecar_description/meshes/right_front_wheel.STL" scale="3 3 3"/>
   </geometry>
 </xacro:macro>
@@ -71,5 +71,5 @@
   <origin xyz="0 0 0" rpy="0 0 0" />
   <geometry>
-    <mesh filename="package://racecar_description/meshes/left_steering_hinge.STL" />
+    <mesh filename="package://racecar_description/meshes/left_steering_hinge.STL" scale="3 3 3"/>
   </geometry>
 </xacro:macro>
@@ -77,17 +77,17 @@
   <origin xyz="0 0 0" rpy="0 0 0" />
   <geometry>
-    <mesh filename="package://racecar_description/meshes/right_steering_hinge.STL" />
+    <mesh filename="package://racecar_description/meshes/right_steering_hinge.STL" scale="3 3 3"/>
   </geometry>
 </xacro:macro>
 <xacro:macro name="left_wheels_collision_geometry">
-  <origin xyz="0 0 -0.0225" rpy="0 0 0" />
+  <origin xyz="0 0 -0.1025" rpy="0 0 0" />
   <geometry>
-    <cylinder length="0.045" radius="0.05" />
+    <cylinder length="0.205" radius="0.25" />
   </geometry>
 </xacro:macro>
 <xacro:macro name="right_wheels_collision_geometry">
-  <origin xyz="0 0 0.0225" rpy="0 0 0" />
+  <origin xyz="0 0 0.1025" rpy="0 0 0" />
   <geometry>
-    <cylinder length="0.045" radius="0.05" />
+    <cylinder length="0.205" radius="0.25" />
   </geometry>
 </xacro:macro>

File: src/simulator/racecar_description/urdf/racecar.xacro (robot description, xacro)
@@ -42,5 +42,5 @@
   </link>
   <joint name="left_rear_wheel_joint" type="continuous">
-    <origin xyz="0 0.1 0" rpy="1.5708 0 0" />
+    <origin xyz="0 0.30 0" rpy="1.5708 0 0" />
     <parent link="chassis" />
     <child link="left_rear_wheel" />
@@ -63,5 +63,5 @@
   </link>
   <joint name="right_rear_wheel_joint" type="continuous">
-    <origin xyz="0 -0.1 0" rpy="1.5708 0 0" />
+    <origin xyz="0 -0.30 0" rpy="1.5708 0 0" />
     <parent link="chassis" />
     <child link="right_rear_wheel" />
@@ -81,5 +81,5 @@
   </link>
   <joint name="left_steering_hinge_joint" type="revolute">
-    <origin xyz="0.325 0.1 0" rpy="0 1.5708 0" />
+    <origin xyz="0.975 0.30 0" rpy="0 1.5708 0" />
     <parent link="chassis" />
     <child link="left_steering_hinge" />
@@ -99,5 +99,5 @@
   </link>
   <joint name="right_steering_hinge_joint" type="continuous">
-    <origin xyz="0.325 -0.1 0" rpy="0 1.5708 0" />
+    <origin xyz="0.975 -0.30 0" rpy="0 1.5708 0" />
     <parent link="chassis" />
     <child link="right_steering_hinge" />
@@ -168,5 +168,5 @@
   </link>
   <joint name="hokuyo_joint" type="fixed">
-    <origin xyz="0.265 0.0 0.075" rpy="0 0 0"/>
+    <origin xyz="0.865 0.0 0.70" rpy="0 0 0"/>
     <parent link="chassis" />
     <child link="laser" />
@@ -176,5 +176,5 @@
   <link name="zed_camera_link">
     <inertial>
-      <mass value="1e-5" />
+      <mass value="5e-5" />
       <origin xyz="0 0 0" rpy="0 0 0"/>
       <inertia ixx="1e-6" ixy="0" ixz="0" iyy="1e-6" iyz="0" izz="1e-6" />
@@ -183,11 +183,11 @@
       <origin xyz="0 0 0" rpy="0 0 0"/>
       <geometry>
-        <box size="0.033 0.175 0.030"/>
-      </geometry>
-    </collision>
-    <visual>
-      <origin xyz="0 0 0" rpy="0 0 0"/>
-      <geometry>
-        <box size="0.033 0.175 0.030"/>
+        <box size="0.065 0.175 0.030"/>
+      </geometry>
+    </collision>
+    <visual>
+      <origin xyz="0 0 0" rpy="0 0 0"/>
+      <geometry>
+        <box size="0.065 0.175 0.030"/>
       </geometry>
       <material name="red"/>
@@ -195,5 +195,5 @@
   </link>
   <joint name="zed_camera_joint" type="fixed">
-    <origin xyz="0.390 0 0.04" rpy="0 0 0"/>
+    <origin xyz="1.0 0 0.20" rpy="0 0 0"/>
     <parent link="chassis"/>
     <child link="zed_camera_link"/>
@@ -205,5 +205,5 @@
   <link name="camera_link"><!-- this needs to match the name in zed_wrapper/zed_tf.launch -->
     <inertial>
-      <mass value="1e-5" />
+      <mass value="5e-5" />
       <origin xyz="0 0 0" rpy="0 0 0"/>
       <inertia ixx="1e-6" ixy="0" ixz="0" iyy="1e-6" iyz="0" izz="1e-6" />
@@ -212,5 +212,5 @@
   <link name="zed_camera_right_link">
     <inertial>
-      <mass value="1e-5" />
+      <mass value="5e-5" />
       <origin xyz="0 0 0" rpy="0 0 0"/>
       <inertia ixx="1e-6" ixy="0" ixz="0" iyy="1e-6" iyz="0" izz="1e-6" />
@@ -218,5 +218,5 @@
   </link>
   <joint name="zed_camera_left_joint" type="fixed">
-    <origin xyz="0 0.06 0" rpy="0 0 0"/>
+    <origin xyz="0 0.30 0" rpy="0 0 0"/>
     <parent link="zed_camera_link"/>
     <child link="camera_link"/>
@@ -224,5 +224,5 @@
   </joint>
   <joint name="zed_camera_right_joint" type="fixed">
-    <origin xyz="0 -0.06 0" rpy="0 0 0"/>
+    <origin xyz="0 -0.30 0" rpy="0 0 0"/>
     <parent link="zed_camera_link"/>
     <child link="zed_camera_right_link"/>

Commit message: ran pre-commit

File: src/simulator/racecar_description/urdf/macros.xacro (robot description, xacro)
@@ -1,3 +1,3 @@
-<?xml version="1.0"?>
+<?xml version="1.0" ?>
 <robot name="racecar" xmlns:xacro="http://www.ros.org/wiki/xacro">
 <!-- inertial parameter macros -->
@@ -5,35 +5,46 @@
   <origin xyz="0.1477 0 0" rpy="0 0 0" />
   <mass value="4.0" />
-  <inertia ixx="0.010609" ixy="0"          ixz="0"
-                          iyy="0.050409"   iyz="0"
-                                           izz="0.05865" />
+  <inertia
+      ixx="0.010609"
+      ixy="0"
+      ixz="0"
+      iyy="0.050409"
+      iyz="0"
+      izz="0.05865"
+    />
 </xacro:macro>
 <xacro:macro name="left_wheels_inertial_params">
   <origin xyz="0 0 -0.0225" rpy="0 0 0" />
   <mass value="0.34055" />
-  <inertia ixx="0.00026046" ixy="0"          ixz="0"
-                            iyy="0.00026046" iyz="0"
-                                             izz="0.00041226" />
+  <inertia
+      ixx="0.00026046"
+      ixy="0"
+      ixz="0"
+      iyy="0.00026046"
+      iyz="0"
+      izz="0.00041226"
+    />
 </xacro:macro>
 <xacro:macro name="right_wheels_inertial_params">
   <origin xyz="0 0 0.0225" rpy="0 0 0" />
   <mass value="0.34055" />
-  <inertia ixx="0.00026046" ixy="0"          ixz="0"
-                            iyy="0.00026046" iyz="0"
-                                             izz="0.00041226" />
+  <inertia
+      ixx="0.00026046"
+      ixy="0"
+      ixz="0"
+      iyy="0.00026046"
+      iyz="0"
+      izz="0.00041226"
+    />
 </xacro:macro>
 <xacro:macro name="steering_hinge_inertial_params">
   <origin xyz="0 0 0" rpy="0 0 0" />
   <mass value="0.100" />
-  <inertia ixx="4E-06" ixy="0"           ixz="0"
-                            iyy="4E-06"  iyz="0"
-                                              izz="4E-06" />
+  <inertia ixx="4E-06" ixy="0" ixz="0" iyy="4E-06" iyz="0" izz="4E-06" />
 </xacro:macro>
 <xacro:macro name="hokuyo_inertial_params">
   <origin xyz="0 0 0" rpy="0 0 0" />
   <mass value="0.130" />
-  <inertia ixx="4E-06" ixy="0"           ixz="0"
-                            iyy="4E-06"  iyz="0"
-                                              izz="4E-06" />
+  <inertia ixx="4E-06" ixy="0" ixz="0" iyy="4E-06" iyz="0" izz="4E-06" />
 </xacro:macro>
 <!-- geometry macros -->
@@ -53,5 +64,7 @@
   <origin xyz="0 0 0" rpy="0 0 0" />
   <geometry>
-    <mesh filename="package://racecar_description/meshes/right_rear_wheel.STL" />
+    <mesh
+        filename="package://racecar_description/meshes/right_rear_wheel.STL"
+      />
   </geometry>
 </xacro:macro>
@@ -59,5 +72,7 @@
   <origin xyz="0 0 0" rpy="0 0 0" />
   <geometry>
-    <mesh filename="package://racecar_description/meshes/left_front_wheel.STL" />
+    <mesh
+        filename="package://racecar_description/meshes/left_front_wheel.STL"
+      />
   </geometry>
 </xacro:macro>
@@ -65,5 +80,7 @@
   <origin xyz="0 0 0" rpy="0 0 0" />
   <geometry>
-    <mesh filename="package://racecar_description/meshes/right_front_wheel.STL" />
+    <mesh
+        filename="package://racecar_description/meshes/right_front_wheel.STL"
+      />
   </geometry>
 </xacro:macro>
@@ -71,5 +88,7 @@
   <origin xyz="0 0 0" rpy="0 0 0" />
   <geometry>
-    <mesh filename="package://racecar_description/meshes/left_steering_hinge.STL" />
+    <mesh
+        filename="package://racecar_description/meshes/left_steering_hinge.STL"
+      />
   </geometry>
 </xacro:macro>
@@ -77,5 +96,7 @@
   <origin xyz="0 0 0" rpy="0 0 0" />
   <geometry>
-    <mesh filename="package://racecar_description/meshes/right_steering_hinge.STL" />
+    <mesh
+        filename="package://racecar_description/meshes/right_steering_hinge.STL"
+      />
   </geometry>
 </xacro:macro>
@@ -97,8 +118,10 @@
     <type>transmission_interface/SimpleTransmission</type>
     <joint name="${name}_joint">
-      <hardwareInterface>hardware_interface/EffortJointInterface</hardwareInterface>
+      <hardwareInterface
+        >hardware_interface/EffortJointInterface</hardwareInterface>
     </joint>
     <actuator name="${name}_motor">
-      <hardwareInterface>hardware_interface/EffortJointInterface</hardwareInterface>
+      <hardwareInterface
+        >hardware_interface/EffortJointInterface</hardwareInterface>
       <mechanicalReduction>1</mechanicalReduction>
     </actuator>
@@ -109,8 +132,10 @@
     <type>transmission_interface/SimpleTransmission</type>
     <joint name="${name}_joint">
-      <hardwareInterface>hardware_interface/EffortJointInterface</hardwareInterface>
+      <hardwareInterface
+        >hardware_interface/EffortJointInterface</hardwareInterface>
     </joint>
     <actuator name="${name}_motor">
-      <hardwareInterface>hardware_interface/EffortJointInterface</hardwareInterface>
+      <hardwareInterface
+        >hardware_interface/EffortJointInterface</hardwareInterface>
       <mechanicalReduction>1</mechanicalReduction>
     </actuator>

File: src/simulator/racecar_description/urdf/materials.xacro (robot description, xacro)
@@ -1,27 +1,27 @@
-<?xml version="1.0"?>
+<?xml version="1.0" ?>
 <robot name="racecar" xmlns:xacro="http://www.ros.org/wiki/xacro">
 <material name="black">
-  <color rgba="0.0 0.0 0.0 1.0"/>
+  <color rgba="0.0 0.0 0.0 1.0" />
 </material>
 <material name="blue">
-  <color rgba="0.0 0.0 0.8 1.0"/>
+  <color rgba="0.0 0.0 0.8 1.0" />
 </material>
 <material name="green">
-  <color rgba="0.0 0.8 0.0 1.0"/>
+  <color rgba="0.0 0.8 0.0 1.0" />
 </material>
 <material name="grey">
-  <color rgba="0.2 0.2 0.2 1.0"/>
+  <color rgba="0.2 0.2 0.2 1.0" />
 </material>
 <material name="orange">
-  <color rgba="${255/255} ${108/255} ${10/255} 1.0"/>
+  <color rgba="${255/255} ${108/255} ${10/255} 1.0" />
 </material>
 <material name="brown">
-  <color rgba="${222/255} ${207/255} ${195/255} 1.0"/>
+  <color rgba="${222/255} ${207/255} ${195/255} 1.0" />
 </material>
 <material name="red">
-  <color rgba="0.8 0.0 0.0 1.0"/>
+  <color rgba="0.8 0.0 0.0 1.0" />
 </material>
 <material name="white">
-  <color rgba="1.0 1.0 1.0 1.0"/>
+  <color rgba="1.0 1.0 1.0 1.0" />
 </material>
 </robot>

File: src/simulator/racecar_description/urdf/racecar.xacro (robot description, xacro)
@@ -1,3 +1,3 @@
-<?xml version="1.0"?>
+<?xml version="1.0" ?>
 <robot name="racecar" xmlns:xacro="http://www.ros.org/wiki/xacro">
   <xacro:include filename="$(find racecar_description)/urdf/macros.xacro" />
@@ -6,9 +6,9 @@
   <link name="chassis">
     <visual>
-      <xacro:chassis_geometry/>
+      <xacro:chassis_geometry />
       <material name="blue" />
     </visual>
     <collision>
-    	<xacro:chassis_geometry/>
+    	<xacro:chassis_geometry />
     </collision>
   </link>
@@ -145,5 +145,5 @@
     <child link="right_front_wheel" />
     <axis xyz="0 0 -1" />
-    <limit effort="10" velocity="100"/>
+    <limit effort="10" velocity="100" />
   </joint>
   <xacro:wheel_transmission name="right_front_wheel" />
@@ -154,13 +154,13 @@
     </inertial>
     <collision>
-      <origin xyz="0 0 0" rpy="0 0 0"/>
-      <geometry>
-        <box size="0.1 0.1 0.1"/>
-      </geometry>
-    </collision>
-    <visual>
-      <origin xyz="0 0 0" rpy="0 0 0"/>
-      <geometry>
-        <mesh filename="package://racecar_description/meshes/hokuyo.dae"/>
+      <origin xyz="0 0 0" rpy="0 0 0" />
+      <geometry>
+        <box size="0.1 0.1 0.1" />
+      </geometry>
+    </collision>
+    <visual>
+      <origin xyz="0 0 0" rpy="0 0 0" />
+      <geometry>
+        <mesh filename="package://racecar_description/meshes/hokuyo.dae" />
         <material name="grey" />
       </geometry>
@@ -168,5 +168,5 @@
   </link>
   <joint name="hokuyo_joint" type="fixed">
-    <origin xyz="0.265 0.0 0.075" rpy="0 0 0"/>
+    <origin xyz="0.265 0.0 0.075" rpy="0 0 0" />
     <parent link="chassis" />
     <child link="laser" />
@@ -177,25 +177,25 @@
     <inertial>
       <mass value="1e-5" />
-      <origin xyz="0 0 0" rpy="0 0 0"/>
+      <origin xyz="0 0 0" rpy="0 0 0" />
       <inertia ixx="1e-6" ixy="0" ixz="0" iyy="1e-6" iyz="0" izz="1e-6" />
     </inertial>
     <collision>
-      <origin xyz="0 0 0" rpy="0 0 0"/>
-      <geometry>
-        <box size="0.033 0.175 0.030"/>
-      </geometry>
-    </collision>
-    <visual>
-      <origin xyz="0 0 0" rpy="0 0 0"/>
-      <geometry>
-        <box size="0.033 0.175 0.030"/>
-      </geometry>
-      <material name="red"/>
+      <origin xyz="0 0 0" rpy="0 0 0" />
+      <geometry>
+        <box size="0.033 0.175 0.030" />
+      </geometry>
+    </collision>
+    <visual>
+      <origin xyz="0 0 0" rpy="0 0 0" />
+      <geometry>
+        <box size="0.033 0.175 0.030" />
+      </geometry>
+      <material name="red" />
     </visual>
   </link>
   <joint name="zed_camera_joint" type="fixed">
-    <origin xyz="0.390 0 0.04" rpy="0 0 0"/>
-    <parent link="chassis"/>
-    <child link="zed_camera_link"/>
+    <origin xyz="0.390 0 0.04" rpy="0 0 0" />
+    <parent link="chassis" />
+    <child link="zed_camera_link" />
     <axis xyz="0 0 1" />
     <!-- <limit lower="0.0" upper="0.0" effort="0.0" velocity="0.0" /> -->
@@ -203,8 +203,10 @@
   <!-- zed camera lenses -->
   <!-- It seems these have to have a non-zero mass to have a camera attached? -->
-  <link name="camera_link"><!-- this needs to match the name in zed_wrapper/zed_tf.launch -->
+  <link
+    name="camera_link"
+  ><!-- this needs to match the name in zed_wrapper/zed_tf.launch -->
     <inertial>
       <mass value="1e-5" />
-      <origin xyz="0 0 0" rpy="0 0 0"/>
+      <origin xyz="0 0 0" rpy="0 0 0" />
       <inertia ixx="1e-6" ixy="0" ixz="0" iyy="1e-6" iyz="0" izz="1e-6" />
     </inertial>
@@ -213,18 +215,18 @@
     <inertial>
       <mass value="1e-5" />
-      <origin xyz="0 0 0" rpy="0 0 0"/>
+      <origin xyz="0 0 0" rpy="0 0 0" />
       <inertia ixx="1e-6" ixy="0" ixz="0" iyy="1e-6" iyz="0" izz="1e-6" />
     </inertial>
   </link>
   <joint name="zed_camera_left_joint" type="fixed">
-    <origin xyz="0 0.06 0" rpy="0 0 0"/>
-    <parent link="zed_camera_link"/>
-    <child link="camera_link"/>
+    <origin xyz="0 0.06 0" rpy="0 0 0" />
+    <parent link="zed_camera_link" />
+    <child link="camera_link" />
     <axis xyz="0 0 1" />
   </joint>
   <joint name="zed_camera_right_joint" type="fixed">
-    <origin xyz="0 -0.06 0" rpy="0 0 0"/>
-    <parent link="zed_camera_link"/>
-    <child link="zed_camera_right_link"/>
+    <origin xyz="0 -0.06 0" rpy="0 0 0" />
+    <parent link="zed_camera_link" />
+    <child link="zed_camera_right_link" />
     <axis xyz="0 0 1" />
   </joint>
